File: hardware/ct-1740-psu-board/ct-1740-psu-board.kicad_pcb (KiCad board)
At the start: 2 copper layers, 170 x 90 mm, 32 parts, among them J1 Conn_01x07, J3 Conn_01x05, P201 Conn_01x06, U1 AQY282EH, U11 Conn_01x03, U12 Conn_01x03, U13 Conn_01x03, U31 LM317, U41 LM317, U51 L78L24

Commit message: Rev. B
Parts:
- added R51: 3.3k, Resistors_THT:R_Axial_DIN0207_L6.3mm_D2.5mm_P10.16mm_Horizontal, F.Cu at (171.8, 67.5)
Connections:
- net ~~20-L renamed ~~20V-L
- net ~~20-N renamed ~~20V-N
- net ~~25-L renamed ~~25V-L
- net ~~25-N renamed ~~25V-N
- net ~~3.3-L renamed ~~3.3V-L
- net ~~3.3-N renamed ~~3.3V-N
