File: hardware/psu-module-positive_BL9342/psu-module-positive.sch (KiCad schematic (older format))
At the start: 15 parts, among them J5 Conn_01x03, U1 BL9342

Commit message: Rev. B
Parts:
- added R4: 100k, Resistors_SMD:R_0805, symbol Device:R_Small
- added R5: 10k, Resistors_SMD:R_0805, symbol Device:R_Small
- R3: value 24k -> 22k; LCSC C17575 -> C17560
Connections:
- net +35V: now also R4.1
- net GND: now also R5.2
- net EN: now reaches U1.4 (~SHDN)
- net EN: now also R4.2, R5.1
Changed lines of the file:
@@
 P 7850 4050
 F 0 "R3" H 7909 4096 50  0000 L CNN
-F 1 "24k" H 7909 4005 50  0000 L CNN
+F 1 "22k" H 7909 4005 50  0000 L CNN
 F 2 "Resistors_SMD:R_0805" H 7850 4050 50  0001 C CNN
 F 3 "~" H 7850 4050 50  0001 C CNN
-F 4 "C17575" H 7850 4050 50  0001 C CNN "LCSC"
+F 4 "C17560" H 7850 4050 50  0001 C CNN "LCSC"
 	1    7850 4050
 	1    0    0    -1
@@
 Wire Wire Line
 	7400 2950 7700 2950
+Text GLabel 5300 2050 0    50   Input ~ 0
+EN
+Text GLabel 5100 3100 0    50   Input ~ 0
+EN
+Text GLabel 5250 2750 1    50   Input ~ 0
++35V
+$Comp
+L Device:R_Small R4
+U 1 1 619FDFA7
+P 5250 2850
+F 0 "R4" H 5309 2896 50  0000 L CNN
+F 1 "100k" H 5309 2805 50  0000 L CNN
+F 2 "Resistors_SMD:R_0805" H 5250 2850 50  0001 C CNN
+F 3 "~" H 5250 2850 50  0001 C CNN
+F 4 "C17407" H 5250 2850 50  0001 C CNN "LCSC"
+	1    5250 2850
+	1    0    0    -1
+$EndComp
+$Comp
+L Device:R_Small R5
+U 1 1 619FED4D
+P 5250 3350
+F 0 "R5" H 5309 3396 50  0000 L CNN
+F 1 "10k" H 5309 3305 50  0000 L CNN
+F 2 "Resistors_SMD:R_0805" H 5250 3350 50  0001 C CNN
+F 3 "~" H 5250 3350 50  0001 C CNN
+F 4 "C17414" H 5250 3350 50  0001 C CNN "LCSC"
+	1    5250 3350
+	1    0    0    -1
+$EndComp
+$Comp
+L power:GND #PWR0109
+U 1 1 619FF309
+P 5250 3450
+F 0 "#PWR0109" H 5250 3200 50  0001 C CNN
+F 1 "GND" H 5250 3300 50  0000 C CNN
+F 2 "" H 5250 3450 50  0001 C CNN
+F 3 "" H 5250 3450 50  0001 C CNN
+	1    5250 3450
+	1    0    0    -1
+$EndComp
+Wire Wire Line
+	5250 2950 5250 3100
+Wire Wire Line
+	5100 3100 5250 3100
+Connection ~ 5250 3100
+Wire Wire Line
+	5250 3100 5250 3250
 $EndSCHEMATC
