File: hardware/psu-module-positive_BL9342/psu-module-positive.kicad_pcb (KiCad board)
At the start: 2 copper layers, 20 x 30 mm, 15 parts, among them J5 Conn_01x03, U1 BL9342

Commit message: Rev. B
Parts:
- added R4: 100k, Resistors_SMD:R_0805, F.Cu at (20.5, 13.8)
- added R5: 10k, Resistors_SMD:R_0805, F.Cu at (17.0, 13.8)
- C3: renamed from C6; value 22µF -> 33pF
- R1: value 100k -> 120k
- R2: value 5.6k -> 6.8k
- R3: value 18k -> 22k
- moved C1 1.60 mm to (17.8, 16.2)
- moved C2 0.75 mm to (18.8, 7.75)
- moved U1 0.75 mm to (18.8, 10.8)
- renumbered C3 to C4, C4 to C5, C5 to C6
Connections:
- U1 pad 4: Net-(U1-Pad4) -> EN
Routing:
- net Net-(C2-Pad2): track 40.2 -> 29.1 mm
- net EN: track 0.00 -> 3.88 mm
- net +35V: track 17.6 -> 18.5 mm
- net FB: track 18.5 -> 19.2 mm
Other:
- board text added: "OR"

Commit message: Rev. C: Hardware
Other:
- board text added: "15V"
- board text added: "5V"
- board text removed: "15"
- board text removed: "5"
- board text removed: "V-SELECTOR"
