File: hardware/cr-17xx-psu-board/cr-17xx-psu-board.kicad_pcb (KiCad board)
At the start: 2 copper layers, 111.5 x 95 mm, 36 parts, among them J1 Conn_01x01, J10 Conn_01x01, J11 Conn_01x01, J12 Conn_01x01, J2 Conn_01x01, J3 Conn_01x01, J4 Conn_01x01, J5 Conn_01x01, J6 Conn_01x01, J7 Conn_01x01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

Commit message: Rev. C: Hardware
Other:
- board text added: "80mAT"
- board text removed: "100mAT"
