File: hardware/psu-module-negative/psu-module-negative.kicad_pcb (KiCad board)
At the start: 2 copper layers, 18 x 30 mm, 8 parts, among them J1 Conn_01x03, U1 MC78L12_TO92, U2 TC7662AxPA

Commit message: Rev. C: Hardware
Parts:
- D1: footprint Diodes_THT:D_DO-35_SOD27_P5.08mm_Vertical_AnodeUp -> Diodes_THT:D_DO-35_SOD27_P7.62mm_Horizontal
Routing:
- net +35V: track 23.5 -> 20.8 mm
- net GND: track 37.8 -> 39.0 mm
