File: hardware/psu-module-negative/psu-module-negative.sch (KiCad schematic (older format))
At the start: 8 parts, among them J1 Conn_01x03, U1 MC78L12_TO92, U2 TC7662AxPA

Commit message: Rev. B
Parts:
- D1: value 4.3V -> 7.5V
Changed lines of the file:
@@
 P 3150 1950
 F 0 "D1" V 3104 2030 50  0000 L CNN
-F 1 "4.3V" V 3195 2030 50  0000 L CNN
+F 1 "7.5V" V 3195 2030 50  0000 L CNN
 F 2 "Diodes_THT:D_DO-35_SOD27_P5.08mm_Vertical_AnodeUp" H 3150 1950 50  0001 C CNN
 F 3 "~" H 3150 1950 50  0001 C CNN

Commit message: Rev. C: Hardware
Parts:
- D1: footprint Diodes_THT:D_DO-35_SOD27_P5.08mm_Vertical_AnodeUp -> Diodes_THT:D_DO-35_SOD27_P7.62mm_Horizontal
Changed lines of the file:
@@
 F 0 "D1" V 3104 2030 50  0000 L CNN
 F 1 "7.5V" V 3195 2030 50  0000 L CNN
-F 2 "Diodes_THT:D_DO-35_SOD27_P5.08mm_Vertical_AnodeUp" H 3150 1950 50  0001 C CNN
+F 2 "Diodes_THT:D_DO-35_SOD27_P7.62mm_Horizontal" H 3150 1950 50  0001 C CNN
 F 3 "~" H 3150 1950 50  0001 C CNN
 	1    3150 1950
