File: hardware/synthesizer-board/synthesizer-board.kicad_pcb (KiCad board)
At the start: 2 copper layers, 154.5 x 127 mm, 171 parts, among them J1 SWD, J11 SELECTOR, J21 SELECTOR, J4 Conn_01x07, J401 SELECTOR, J751 SELECTOR, P601 Conn_01x06_Male, P602 Conn_01x16_Male, P603 Conn_01x14_Male, P604 Conn_01x06_Male, Q101 BC847, Q201 BC847, Q301 BC847, Q401 BC847, Q701 BC847, Q702 BC847, Q703 BC847, Q704 BC847, Q705 BC847, Q721 BC847, Q731 BC847, Q741 BC847, Q751 BC847, Q811 BC847, Q821 BC847, Q831 BC847, Q841 BC847, Q851 BC847, Q861 BC847, Q871 BC847, U1 STM32G070RBTx, U101 U813, U11 BL9342, U21 BL9342, U601 TLP291-4GB, U602 TLP291-4GB, U603 TLP291-4GB, U604 TLP291GB, U605 AQY282SX, Y1 16MHz, Y2 32.768kHz

Commit message: Rev. B
Parts:
- removed J401: SELECTOR, Pin_Headers:Pin_Header_Straight_1x03_Pitch2.54mm
- added C11: 1nF, Capacitors_SMD:C_0805, F.Cu at (183.0, 144.0)
- added C18: 1nF, Capacitors_SMD:C_0805, F.Cu at (176.5, 112.0)
- added C21: 1nF, Capacitors_SMD:C_0805, F.Cu at (208.2, 142.5)
- added C28: 1nF, Capacitors_SMD:C_0805, F.Cu at (210.6, 112.0)
- added J10: Conn_01x01, Measurement_Points:Measurement_Point_Round-TH_Small, F.Cu at (213.8, 138.6)
- added J12: Conn_01x01, Measurement_Points:Measurement_Point_Round-TH_Small, F.Cu at (194.0, 44.0)
- added J13: Conn_01x01, Measurement_Points:Measurement_Point_Round-TH_Small, F.Cu at (181.8, 40.5)
- added J14: Conn_01x01, Measurement_Points:Measurement_Point_Round-TH_Small, F.Cu at (207.0, 44.0)
- added J15: Conn_01x01, Measurement_Points:Measurement_Point_Round-TH_Small, F.Cu at (96.5, 139.0)
- added J16: Conn_01x01, Measurement_Points:Measurement_Point_Round-TH_Small, F.Cu at (170.5, 75.5)
- added J17: Conn_01x01, Measurement_Points:Measurement_Point_Round-TH_Small, F.Cu at (216.0, 68.1)
- added J18: Conn_01x01, Measurement_Points:Measurement_Point_Round-TH_Small, F.Cu at (200.5, 74.0)
- added J19: Conn_01x01, Measurement_Points:Measurement_Point_Round-TH_Small, F.Cu at (196.5, 74.0)
- added J2: Conn_01x01, Measurement_Points:Measurement_Point_Round-TH_Small, F.Cu at (180.0, 112.0)
- added J20: Conn_01x01, Measurement_Points:Measurement_Point_Round-TH_Small, F.Cu at (174.5, 63.5)
- added J22: Conn_01x01, Measurement_Points:Measurement_Point_Round-TH_Small, F.Cu at (151.5, 113.1)
- added J23: Conn_01x01, Measurement_Points:Measurement_Point_Round-TH_Small, F.Cu at (156.5, 113.1)
- added J3: Conn_01x01, Measurement_Points:Measurement_Point_Round-TH_Small, F.Cu at (207.1, 112.0)
- added J5: Conn_01x01, Measurement_Points:Measurement_Point_Round-TH_Small, F.Cu at (185.5, 143.0)
- added J6: Conn_01x01, Measurement_Points:Measurement_Point_Round-TH_Small, F.Cu at (210.8, 141.5)
- added J7: Conn_01x01, Measurement_Points:Measurement_Point_Round-TH_Small, F.Cu at (173.2, 115.0)
- added J8: Conn_01x01, Measurement_Points:Measurement_Point_Round-TH_Small, F.Cu at (213.8, 115.0)
- added J9: Conn_01x01, Measurement_Points:Measurement_Point_Round-TH_Small, F.Cu at (173.2, 138.6)
- J11, J21: value SELECTOR -> Conn_01x01; footprint Pin_Headers:Pin_Header_Straight_1x03_Pitch2.54mm -> Measurement_Points:Measurement_Point_Round-TH_Small
- P603: value Conn_01x14_Male -> JST NH
- P604: value Conn_01x06_Male -> JST NH
- R11, R21: value 120k -> 33k
- R12: value 39k -> 10k
- R22: value 24k -> 6.2k
- R721, R731: value 3.3k -> 33k
- U11, U21: value BL9342 -> LV2841XL
- U601, U602, U603: value TLP291-4GB -> LTV-247
- U604: value TLP291GB -> LTV-217
- moved J11 93.3 mm to (167.6, 44.0), turned to 0 degrees
- moved J21 67.6 mm to (146.5, 113.1), turned to 0 degrees
- moved D401 10.3 mm to (196.5, 69.0)
- moved R403 10.3 mm to (196.5, 64.5)
- moved Q401 7.07 mm to (205.5, 64.5)
- moved R401 7.07 mm to (200.5, 69.0)
- moved R402 7.07 mm to (200.5, 64.5)
- moved C12 3.01 mm to (186.5, 131.8)
- moved C13 3.01 mm to (180.0, 128.2)
- moved C14 3.01 mm to (175.0, 131.8)
- moved C15 3.01 mm to (185.0, 122.2)
- moved C16 3.01 mm to (187.5, 122.2)
- moved C17 3.01 mm to (190.0, 122.2)
- moved D11 3.01 mm to (187.5, 128.2)
- moved L11 3.01 mm to (180.0, 123.2)
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- renumbered C11 to C12, C12 to C13, C13 to C14, C14 to C15, C15 to C16, C16 to C17, C21 to C22, C22 to C23, C23 to C24, C24 to C25, C25 to C26, C26 to C27
Connections:
- C12 pad 1: Net-(C11-Pad1) -> +5V|+15V
- C22 pad 1: Net-(C21-Pad1) -> +15V
- D401 pad 2: MUTING -> MUTING_B
- J11 pad 1: +15V -> FM_FREQUENCY
- J21 pad 1: +15V -> MANUAL
- R401 pad 1: MUTING -> MUTING_A
- R402 pad 2: Net-(J401-Pad1) -> J601_5
- R403 pad 2: Net-(J401-Pad3) -> J601_5
- U1 pad 14: MUTING -> MUTING_A
- U1 pad 16: Net-(U1-Pad16) -> MUTING_B
- U11 pad 5: Net-(C11-Pad1) -> +5V|+15V
- U21 pad 5: Net-(C21-Pad1) -> +15V
Routing:
- net MUTING: track 70.3 -> 0.00 mm
- net MUTING_A: track 0.00 -> 70.1 mm
- net MUTING_B: track 0.00 -> 64.0 mm, vias 0 -> 2
- net GND: track 104.3 -> 140.0 mm, vias 208 -> 176
- net +5V|+15V: track 59.2 -> 30.9 mm, vias 2 -> 1
- net +3V3: track 350.4 -> 368.2 mm, vias 6 -> 3
- net Net-(C21-Pad1): track 8.69 -> 0.00 mm
- net Net-(C11-Pad1): track 8.69 -> 0.00 mm
- net Net-(C104-Pad2): track 7.14 -> 13.7 mm
- net Net-(J401-Pad3): track 5.07 -> 0.00 mm
- net Net-(J401-Pad1): track 5.07 -> 0.00 mm
- net +15V: track 145.1 -> 150.1 mm, vias 3 -> 2
- net Net-(C201-Pad2): track 6.96 -> 11.0 mm
- net TUNING_VOLTAGE: track 37.6 -> 41.6 mm
- net Net-(C303-Pad2): track 8.04 -> 12.0 mm
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Other:
- board text added: "1Vpp"
- board text added: "500mVpp"
- board text added: "5Vpp"
- board text added: "JUMPER A: CR-1750 + CR-1780 SN: < 20.000 JUMPER B: CR-1750 + CR-1780 SN: > 20.000 / CT-1740"
- board text added: "Rev. B 2021-11-27 Yannick Bock dual-board.de"
- board text removed: "JUMPER A: CR-1750 / CR-1780 SN: < 20.000 JUMPER B: CR-1750 / CR-1780 SN: > 20.000 / CT-1740"
- board text removed: "Rev. A 2021-11-13 Yannick Bock dual-board.de"

Commit message: Rev. C: Hardware
Parts:
- added J24: RESERVE, Pin_Headers:Pin_Header_Straight_2x06_Pitch2.54mm, F.Cu at (102.5, 94.8)
- moved J1 6.00 mm to (121.5, 70.0)
Connections:
- U1 pad 18: Net-(U1-Pad18) -> RES_PA1
- U1 pad 19: Net-(U1-Pad19) -> RES_PA2
- U1 pad 20: Net-(U1-Pad20) -> RES_PA3
- U1 pad 21: Net-(U1-Pad21) -> RES_PA4
- U1 pad 22: Net-(U1-Pad22) -> RES_PA5
- U1 pad 30: Net-(U1-Pad30) -> RES_PB10
- U1 pad 31: Net-(U1-Pad31) -> RES_PB11
Routing:
- net +5V: track 170.7 -> 284.5 mm, vias 5 -> 7
- net RES_PA5: track 0.00 -> 96.0 mm, vias 0 -> 2
- net RES_PA4: track 0.00 -> 93.7 mm, vias 0 -> 2
- net RES_PA3: track 0.00 -> 91.5 mm, vias 0 -> 2
- net RES_PA2: track 0.00 -> 89.2 mm, vias 0 -> 2
- net RES_PA1: track 0.00 -> 86.9 mm, vias 0 -> 2
- net RES_PB11: track 0.00 -> 34.2 mm
- net RES_PB10: track 0.00 -> 30.5 mm
- net +3V3: track 368.2 -> 390.9 mm, vias 3 -> 5
- net DISPLAY_D4: track 45.9 -> 43.4 mm
- net DISPLAY_D3: track 44.2 -> 41.8 mm
- net DISPLAY_D2: track 42.6 -> 40.1 mm
- net DISPLAY_DP: track 38.1 -> 35.6 mm
- net DISPLAY_ON: track 36.5 -> 34.0 mm
- net DISPLAY_D1: track 41.0 -> 38.5 mm
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Other:
- board text added: "5V"
- board text added: "PA1"
- board text added: "PA2"
- board text added: "PA3"
- board text added: "PA4"
- board text added: "PA5"
- board text added: "PB10"
- board text added: "PB11"
- board text added: "Rev. C 2022-01-04 Yannick Bock dual-board.de"
- board text removed: "Rev. B 2021-11-27 Yannick Bock dual-board.de"
