File: hardware/synthesizer-board/synthesizer-board.sch (KiCad schematic (older format))
At the start: 171 parts, among them J1 SWD, J11 SELECTOR, J21 SELECTOR, J4 Conn_01x07, J401 SELECTOR, J751 SELECTOR, P601 Conn_01x06_Male, P602 Conn_01x16_Male, P603 Conn_01x14_Male, P604 Conn_01x06_Male, Q101 BC847, Q201 BC847, Q301 BC847, Q401 BC847, Q701 BC847, Q702 BC847, Q703 BC847, Q704 BC847, Q705 BC847, Q721 BC847, Q731 BC847, Q741 BC847, Q751 BC847, Q811 BC847, Q821 BC847, Q831 BC847, Q841 BC847, Q851 BC847, Q861 BC847, Q871 BC847, U1 STM32G070RBTx, U101 U813, U11 BL9342, U21 BL9342, U601 LTV-247, U602 LTV-247, U603 LTV-247, U604 LTV-217, U605 AQY282SX, Y1 16MHz, Y2 32.768kHz

Commit message: Rev. B
Parts:
- removed J11, J21, J401: SELECTOR, Pin_Headers:Pin_Header_Straight_1x03_Pitch2.54mm, symbol Connector_Generic:Conn_01x03
- added C11, C18, C21, C28: 1nF, Capacitors_SMD:C_0805, symbol Device:C
- added J10, J11, J12, J13, J14, J15, J16, J17, J18, J19, J2, J20, J21, J22, J23, J3, J5, J6, J7, J8, J9: Conn_01x01, Measurement_Points:Measurement_Point_Round-TH_Small, symbol Connector_Generic:Conn_01x01
- P603: value Conn_01x14_Male -> JST NH
- P604: value Conn_01x06_Male -> JST NH
- R11, R21: value 120k -> 33k; LCSC C17436 -> C17633
- R12: value 39k -> 10k; LCSC C25826 -> C17414
- R22: value 24k -> 6.2k; LCSC C17575 -> C17767
- R721, R731: value 3.3k -> 33k; LCSC C26010 -> C17633
- U11, U21: value BL9342 -> LV2841XL; LCSC C93176 -> C225807
- renumbered C11 to C12, C12 to C13, C13 to C14, C14 to C15, C15 to C16, C16 to C17, C21 to C22, C22 to C23, C23 to C24, C24 to C25, C25 to C26, C26 to C27
Connections:
- net +15V: now also C22.1, U21.5 (VIN), C21.2, J6.1 (Pin_1)
- net +3V3: now also C18.1, J2.1 (Pin_1)
- net +5V: now also C28.1, J3.1 (Pin_1)
- net +5V|+15V: now also C12.1, U11.5 (VIN), C11.2, J5.1 (Pin_1)
- net -18V: now also J15.1 (Pin_1)
- net AM_FREQUENCY: now also J12.1 (Pin_1)
- net FM: now also J22.1 (Pin_1)
- net FM_FREQUENCY: now also J11.1 (Pin_1)
- net GND: now also C11.1, C18.2, C21.1, C28.2, J10.1 (Pin_1), J7.1 (Pin_1), J8.1 (Pin_1), J9.1 (Pin_1)
- net J601_5: now also R402.2, R403.2
- net MANUAL: now also J21.1 (Pin_1)
- net SCAN_STOP: now also J17.1 (Pin_1)
- net STANDBY: now also J23.1 (Pin_1)
- net TUNING_VOLTAGE: now also J16.1 (Pin_1)
- net at C104.2, Q101.1 (B), R101.1: now also J13.1 (Pin_1)
- net at C201.2, Q201.1 (B), R201.1: now also J14.1 (Pin_1)
- net at C303.2, Q301.1 (B), R305.2: now also J20.1 (Pin_1)
- net MUTING_B: now reaches U1.16 (PC3)
- net MUTING_B: now also D401.2 (A), J19.1 (Pin_1)
- net MUTING renamed MUTING_A
- net MUTING_A: now also J18.1 (Pin_1); no longer D401.2 (A)
Other:
- note added: "1Vpp"
- note added: "500mVpp"
- note added: "5Vpp"
- note added: "U11 + U21:\nLMR14006X (LCSC: C478074)\nLV2841XL (LCSC: C225807)"
- note removed: "U11 + U21: LMR14006X (LCSC: C478074)\nR11 + R21: 33k (LCSC: C17633)\nR12: 10k (LCSC: C17414)\nR22: 6.2k (LCSC: C17767)"
- moved on the sheet: C12, C13, C14, C15, C16, C17, C22, C23, C24, C25, C26, C27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

Commit message: Rev. C: Hardware
Parts:
- added J24: RESERVE, Pin_Headers:Pin_Header_Straight_2x06_Pitch2.54mm, symbol Connector_Generic:Conn_02x06_Odd_Even
Connections:
- net +3V3: now also J24.1 (Pin_1)
- net +5V: now also J24.5 (Pin_5)
- net GND: now also J24.3 (Pin_3), J24.7 (Pin_7)
- net RES_PA1: now reaches U1.18 (PA1)
- net RES_PA1: now also J24.10 (Pin_10)
- net RES_PA2: now reaches U1.19 (PA2)
- net RES_PA2: now also J24.8 (Pin_8)
- net RES_PA3: now reaches U1.20 (PA3)
- net RES_PA3: now also J24.6 (Pin_6)
- net RES_PA4: now reaches U1.21 (PA4)
- net RES_PA4: now also J24.4 (Pin_4)
- net RES_PA5: now reaches U1.22 (PA5)
- net RES_PA5: now also J24.2 (Pin_2)
- net RES_PB10: now reaches U1.30 (PB10)
- net RES_PB10: now also J24.11 (Pin_11)
- net RES_PB11: now reaches U1.31 (PB11)
- net RES_PB11: now also J24.9 (Pin_9)
Changed lines of the file:
@@
 	22400 13950 22250 13950
 Connection ~ 22250 13950
+Text GLabel 4950 2250 2    50   BiDi ~ 0
+RES_PA1
+Text GLabel 4950 2350 2    50   BiDi ~ 0
+RES_PA2
+Text GLabel 4950 2450 2    50   BiDi ~ 0
+RES_PA3
+Text GLabel 4950 2550 2    50   BiDi ~ 0
+RES_PA4
+Text GLabel 4950 2650 2    50   BiDi ~ 0
+RES_PA5
+Text GLabel 4950 4850 2    50   BiDi ~ 0
+RES_PB10
+Text GLabel 4950 4950 2    50   BiDi ~ 0
+RES_PB11
+$Comp
+L Connector_Generic:Conn_02x06_Odd_Even J24
+U 1 1 622574A8
+P 6950 4200
+F 0 "J24" V 7167 4196 50  0001 C CNN
+F 1 "RESERVE" H 7000 4525 50  0000 C CNN
+F 2 "Pin_Headers:Pin_Header_Straight_2x06_Pitch2.54mm" H 6950 4200 50  0001 C CNN
+F 3 "~" H 6950 4200 50  0001 C CNN
+	1    6950 4200
+	1    0    0    -1
+$EndComp
+Text GLabel 7250 4400 2    50   BiDi ~ 0
+RES_PA1
+Text GLabel 7250 4300 2    50   BiDi ~ 0
+RES_PA2
+Text GLabel 7250 4200 2    50   BiDi ~ 0
+RES_PA3
+Text GLabel 7250 4100 2    50   BiDi ~ 0
+RES_PA4
+Text GLabel 7250 4000 2    50   BiDi ~ 0
+RES_PA5
+Text GLabel 6750 4500 0    50   BiDi ~ 0
+RES_PB10
+Text GLabel 6750 4400 0    50   BiDi ~ 0
+RES_PB11
+$Comp
+L power:+3.3V #PWR0164
+U 1 1 622994F9
+P 6750 4000
+F 0 "#PWR0164" H 6750 3850 50  0001 C CNN
+F 1 "+3.3V" V 6750 4250 50  0000 C CNN
+F 2 "" H 6750 4000 50  0001 C CNN
+F 3 "" H 6750 4000 50  0001 C CNN
+	1    6750 4000
+	0    -1   -1   0
+$EndComp
+$Comp
+L power:GND #PWR0165
+U 1 1 6229AF13
+P 6750 4300
+F 0 "#PWR0165" H 6750 4050 50  0001 C CNN
+F 1 "GND" V 6750 4100 50  0000 C CNN
+F 2 "" H 6750 4300 50  0001 C CNN
+F 3 "" H 6750 4300 50  0001 C CNN
+	1    6750 4300
+	0    1    1    0
+$EndComp
+$Comp
+L power:+5V #PWR0166
+U 1 1 6229AF1D
+P 6750 4200
+F 0 "#PWR0166" H 6750 4050 50  0001 C CNN
+F 1 "+5V" V 6750 4400 50  0000 C CNN
+F 2 "" H 6750 4200 50  0001 C CNN
+F 3 "" H 6750 4200 50  0001 C CNN
+	1    6750 4200
+	0    -1   -1   0
+$EndComp
+$Comp
+L power:GND #PWR0167
+U 1 1 6229AF27
+P 6750 4100
+F 0 "#PWR0167" H 6750 3850 50  0001 C CNN
+F 1 "GND" V 6750 3900 50  0000 C CNN
+F 2 "" H 6750 4100 50  0001 C CNN
+F 3 "" H 6750 4100 50  0001 C CNN
+	1    6750 4100
+	0    1    1    0
+$EndComp
 $EndSCHEMATC
